Commit message: algunos cambios para agregar la imu, no funciona

File: cartographer_ros/urdf/backpack_2d.urdf (robot description, URDF)
Before this commit: robot cartographer_backpack_2d, 4 links, 3 joints
Links:
- removed link horizontal_laser_link
- removed link imu_link
- removed link vertical_laser_link
- added link laser; visual cylinder length=0.05 radius=0.03
Joints:
- removed joint horizontal_laser_link_joint
- removed joint imu_link_joint
- removed joint vertical_laser_link_joint
- added joint laser_link_joint: type fixed, parent base_link, child laser, origin xyz=0 -0.5 -0.5 rpy=0 0 -1.570796
